Commit message: added camera link and corresponding joint

File: src/udacity_bot/urdf/udacity_bot.xacro (robot description, xacro)
@@ -61,4 +61,28 @@
       <joint_properties damping="1.0" friction="1.0"/>
   </joint>
+	<link name='camera'>
+        <inertial>
+            <mass value="0.1"/>
+            <origin xyz="0.0 0 0" rpy=" 0 0 0"/>
+            <inertia ixx="1e-6" ixy="0" ixz="0" iyy="1e-6" iyz="0" izz="1e-6"/>
+        </inertial>
+        <collision name='collision'>
+            <origin xyz="0.0 0 0" rpy=" 0 0 0"/>
+            <geometry>
+                <box size="0.05 0.05 0.05"/>
+            </geometry>
+        </collision>
+        <visual name='camera_visual'>
+            <origin xyz="0.0 0 0" rpy=" 0 0 0"/>
+            <geometry>
+                <box size="0.05 0.05 0.05"/>
+            </geometry>
+        </visual>
+    </link>
+    <joint type="fixed" name="camera_joint">
+        <origin xyz="0.2 0 0" rpy="0 0 0"/>
+        <child link="camera"/>
+        <parent link="chassis"/>
+    </joint>
   <link name='chassis'>
     <pose>0 0 0.1 0 0 0</pose>

Commit message: hokuyo laser range finder added to robot

File: src/udacity_bot/urdf/udacity_bot.xacro (robot description, xacro)
@@ -7,4 +7,5 @@
     <child link="chassis" />
   </joint>
+<!-- Left wheel -->
 	<link name='left_wheel'>
       <inertial>
@@ -34,4 +35,5 @@
       <joint_properties damping="1.0" friction="1.0"/>
   </joint>
+<!-- Right wheel -->
   <link name='right_wheel'>
       <inertial>
@@ -61,4 +63,5 @@
       <joint_properties damping="1.0" friction="1.0"/>
   </joint>
+<!-- Camera link and joint -->
 	<link name='camera'>
         <inertial>
@@ -80,9 +83,36 @@
         </visual>
     </link>
-    <joint type="fixed" name="camera_joint">
-        <origin xyz="0.2 0 0" rpy="0 0 0"/>
-        <child link="camera"/>
-        <parent link="chassis"/>
-    </joint>
+  <joint type="fixed" name="camera_joint">
+      <origin xyz="0.2 0 0" rpy="0 0 0"/>
+      <child link="camera"/>
+      <parent link="chassis"/>
+  </joint>
+<!--Laser range finder : Hokuyo rangefinder -->
+	<link name='hokuyo'>
+        <inertial>
+            <mass value="0.1"/>
+            <origin xyz="0.0 0 0" rpy=" 0 0 0"/>
+            <inertia ixx="1e-6" ixy="0" ixz="0" iyy="1e-6" iyz="0" izz="1e-6"/>
+        </inertial>
+        <collision name='collision'>
+            <origin xyz="0.0 0 0" rpy=" 0 0 0"/>
+            <geometry>
+                <box size="0.1 0.1 0.1"/>
+            </geometry>
+        </collision>
+        <visual name='hokuyo_visual'>
+            <origin xyz="0.0 0 0" rpy=" 0 0 0"/>
+            <geometry>
+                <mesh filename="package://udacity_bot/meshes/hokuyo.dae"/>
+                <!-- <box size="0.1 0.1 0.1"/> -->
+            </geometry>
+        </visual>
+    </link>
+  <joint type="fixed" name="hokuyo_joint">
+      <origin xyz="0.15 0 0.1" rpy="0 0 0"/>
+      <child link="hokuyo"/>
+      <parent link="chassis"/>
+  </joint>
+<!-- Main robot body including the caster wheels -->
   <link name='chassis'>
     <pose>0 0 0.1 0 0 0</pose>

Commit message: minor mods

File: src/udacity_bot/urdf/udacity_bot.xacro (robot description, xacro)
@@ -1,71 +1,66 @@
 <?xml version='1.0'?>
 <robot name="udacity_bot" xmlns:xacro="http://www.ros.org/wiki/xacro">
-	<!-- Make sure the xacro model loads all the Plugins (differential controller, camera, hokuyo laser scanner) for the gazebo model-->
-	<xacro:include filename="$(find udacity_bot)/urdf/udacity_bot.gazebo" />
-	<!-- init the robot footprint -->
-  <link name="robot_footprint"></link>
-  <joint name="robot_footprint_joint" type="fixed">
-    <origin xyz="0 0 0" rpy="0 0 0" />
-    <parent link="robot_footprint"/>
-    <child link="chassis" />
-  </joint>
-<!-- Left wheel -->
-	<link name='left_wheel'>
-      <inertial>
-          <mass value="5.0"/>
-          <origin xyz="0.0 0 0" rpy=" 0 1.5707 1.5707"/>
-          <inertia ixx="0.1" ixy="0" ixz="0" iyy="0.1" iyz="0" izz="0.1"/>
-      </inertial>
-      <collision name='collision'>
-          <origin xyz="0.0 0 0" rpy=" 0 1.5707 1.5707"/>
-          <geometry>
-              <cylinder length="0.05" radius="0.1"/>
-          </geometry>
-      </collision>
-      <visual name='wheel_visual'>
-          <origin xyz="0.0 0 0" rpy=" 0 1.5707 1.5707"/>
-          <geometry>
-              <cylinder length="0.05" radius="0.1"/>
-          </geometry>
-      </visual>
-  </link>
-  <joint type="continuous" name="left_wheel_hinge">
-      <origin xyz="0 0.15 0" rpy="0 0 0"/>
-      <child link="left_wheel"/>
-      <parent link="chassis"/>
-      <axis xyz="0 1 0" rpy="0 0 0"/>
-      <limit effort="10000" velocity="1000"/>
-      <joint_properties damping="1.0" friction="1.0"/>
-  </joint>
-<!-- Right wheel -->
-  <link name='right_wheel'>
-      <inertial>
-          <mass value="5.0"/>
-          <origin xyz="0.0 0 0" rpy=" 0 1.5707 1.5707"/>
-          <inertia ixx="0.1" ixy="0" ixz="0" iyy="0.1" iyz="0" izz="0.1"/>
-      </inertial>
-      <collision name='collision'>
-          <origin xyz="0.0 0 0" rpy=" 0 1.5707 1.5707"/>
-          <geometry>
-              <cylinder length="0.05" radius="0.1"/>
-          </geometry>
-      </collision>
-      <visual name='wheel_visual'>
-          <origin xyz="0.0 0 0" rpy=" 0 1.5707 1.5707"/>
-          <geometry>
-              <cylinder length="0.05" radius="0.1"/>
-          </geometry>
-      </visual>
-  </link>
-  <joint type="continuous" name="right_wheel_hinge">
-      <origin xyz="0 -0.15 0" rpy="0 0 0"/>
-      <child link="right_wheel"/>
-      <parent link="chassis"/>
-      <axis xyz="0 1 0" rpy="0 0 0"/>
-      <limit effort="10000" velocity="1000"/>
-      <joint_properties damping="1.0" friction="1.0"/>
-  </joint>
-<!-- Camera link and joint -->
-	<link name='camera'>
+    <xacro:include filename="$(find udacity_bot)/urdf/udacity_bot.gazebo" />
+    <link name="robot_footprint"></link>
+    <joint name="robot_footprint_joint" type="fixed">
+        <origin xyz="0 0 0" rpy="0 0 0"/>
+        <parent link="robot_footprint"/>
+        <child link="chassis"/>
+    </joint>
+    <link name='left_wheel'>
+        <inertial>
+            <mass value="5.0"/>
+            <origin xyz="0.0 0 0" rpy=" 0 1.5707 1.5707"/>
+            <inertia ixx="0.1" ixy="0" ixz="0" iyy="0.1" iyz="0" izz="0.1"/>
+        </inertial>
+        <collision name='collision'>
+            <origin xyz="0.0 0 0" rpy=" 0 1.5707 1.5707"/>
+            <geometry>
+                <cylinder length="0.05" radius="0.1"/>
+            </geometry>
+        </collision>
+        <visual name='wheel_visual'>
+            <origin xyz="0.0 0 0" rpy=" 0 1.5707 1.5707"/>
+            <geometry>
+                <cylinder length="0.05" radius="0.1"/>
+            </geometry>
+        </visual>
+    </link>
+    <joint type="continuous" name="left_wheel_hinge">
+        <origin xyz="0 0.15 0" rpy="0 0 0"/>
+        <child link="left_wheel"/>
+        <parent link="chassis"/>
+        <axis xyz="0 1 0" rpy="0 0 0"/>
+        <limit effort="10000" velocity="1000"/>
+        <joint_properties damping="1.0" friction="1.0"/>
+    </joint>
+    <link name='right_wheel'>
+        <inertial>
+            <mass value="5.0"/>
+            <origin xyz="0.0 0 0" rpy=" 0 1.5707 1.5707"/>
+            <inertia ixx="0.1" ixy="0" ixz="0" iyy="0.1" iyz="0" izz="0.1"/>
+        </inertial>
+        <collision name='collision'>
+            <origin xyz="0.0 0 0" rpy=" 0 1.5707 1.5707"/>
+            <geometry>
+                <cylinder length="0.05" radius="0.1"/>
+            </geometry>
+        </collision>
+        <visual name='wheel_visual'>
+            <origin xyz="0.0 0 0" rpy=" 0 1.5707 1.5707"/>
+            <geometry>
+                <cylinder length="0.05" radius="0.1"/>
+            </geometry>
+        </visual>
+    </link>
+    <joint type="continuous" name="right_wheel_hinge">
+        <origin xyz="0 -0.15 0" rpy="0 0 0"/>
+        <child link="right_wheel"/>
+        <parent link="chassis"/>
+        <axis xyz="0 1 0" rpy="0 0 0"/>
+        <limit effort="10000" velocity="1000"/>
+        <joint_properties damping="1.0" friction="1.0"/>
+    </joint>
+    <link name='camera'>
         <inertial>
             <mass value="0.1"/>
@@ -86,11 +81,10 @@
         </visual>
     </link>
-  <joint type="fixed" name="camera_joint">
-      <origin xyz="0.2 0 0" rpy="0 0 0"/>
-      <child link="camera"/>
-      <parent link="chassis"/>
-  </joint>
-<!--Laser range finder : Hokuyo rangefinder -->
-	<link name='hokuyo'>
+    <joint type="fixed" name="camera_joint">
+        <origin xyz="0.2 0 0" rpy="0 0 0"/>
+        <child link="camera"/>
+        <parent link="chassis"/>
+    </joint>
+    <link name='hokuyo'>
         <inertial>
             <mass value="0.1"/>
@@ -112,77 +106,72 @@
         </visual>
     </link>
-  <joint type="fixed" name="hokuyo_joint">
-      <origin xyz="0.15 0 0.1" rpy="0 0 0"/>
-      <child link="hokuyo"/>
-      <parent link="chassis"/>
-  </joint>
-<!-- Main robot body including the caster wheels -->
-  <link name='chassis'>
-    <pose>0 0 0.1 0 0 0</pose>
-    <inertial>
-      <mass value="15.0"/>
-      <origin xyz="0.0 0 0" rpy=" 0 0 0"/>
-      <inertia
-          ixx="0.1" ixy="0" ixz="0"
-          iyy="0.1" iyz="0"
-          izz="0.1"
-      />
-    </inertial>
-    <collision name='collision'>
-      <origin xyz="0 0 0" rpy=" 0 0 0"/>
-      <geometry>
-        <box size=".4 .2 .1"/>
-      </geometry>
-    </collision>
-    <visual name='chassis_visual'>
-      <origin xyz="0 0 0" rpy=" 0 0 0"/>
-      <geometry>
-        <box size=".4 .2 .1"/>
-      </geometry>
-    </visual>
-    <collision name='back_caster_collision'>
-      <origin xyz="-0.15 0 -0.05" rpy=" 0 0 0"/>
-      <geometry>
-        <sphere radius="0.05"/>
-      </geometry>
-      <surface>
-        <friction>
-          <ode>
-            <mu>0</mu>
-            <mu2>0</mu2>
-            <slip1>1.0</slip1>
-            <slip2>1.0</slip2>
-          </ode>
-        </friction>
-      </surface>
-    </collision>
-    <visual name='back_caster_visual'>
-      <origin xyz="-0.15 0 -0.05" rpy=" 0 0 0"/>
-      <geometry>
-        <sphere radius="0.05"/>
-      </geometry>
-    </visual>
-    <collision name='front_caster_collision'>
-      <origin xyz="0.15 0 -0.05" rpy=" 0 0 0"/>
-      <geometry>
-        <sphere radius="0.05"/>
-      </geometry>
-      <surface>
-        <friction>
-          <ode>
-            <mu>0</mu>
-            <mu2>0</mu2>
-            <slip1>1.0</slip1>
-            <slip2>1.0</slip2>
-          </ode>
-        </friction>
-      </surface>
-    </collision>
-    <visual name='front_caster_visual'>
-      <origin xyz="0.15 0 -0.05" rpy=" 0 0 0"/>
-      <geometry>
-        <sphere radius="0.05"/>
-      </geometry>
-    </visual>
-  </link>
+    <joint type="fixed" name="hokuyo_joint">
+        <origin xyz="0.15 0 0.1" rpy="0 0 0"/>
+        <child link="hokuyo"/>
+        <parent link="chassis"/>
+    </joint>
+    <link name='chassis'>
+        <pose>0 0 0.1 0 0 0</pose>
+        <inertial>
+            <mass value="15.0"/>
+            <origin xyz="0.0 0 0" rpy=" 0 0 0"/>
+            <inertia ixx="0.1" ixy="0" ixz="0" iyy="0.1" iyz="0" izz="0.1"/>
+        </inertial>
+        <collision name='collision'>
+            <origin xyz="0 0 0" rpy=" 0 0 0"/>
+            <geometry>
+                <box size=".4 .2 .1"/>
+            </geometry>
+        </collision>
+        <visual name='chassis_visual'>
+            <origin xyz="0 0 0" rpy=" 0 0 0"/>
+            <geometry>
+                <box size=".4 .2 .1"/>
+            </geometry>
+        </visual>
+        <collision name='back_caster_collision'>
+            <origin xyz="-0.15 0 -0.05" rpy=" 0 0 0"/>
+            <geometry>
+                <sphere radius="0.05"/>
+            </geometry>
+            <surface>
+                <friction>
+                    <ode>
+                        <mu>0</mu>
+                        <mu2>0</mu2>
+                        <slip1>1.0</slip1>
+                        <slip2>1.0</slip2>
+                    </ode>
+                </friction>
+            </surface>
+        </collision>
+        <visual name='back_caster_visual'>
+            <origin xyz="-0.15 0 -0.05" rpy=" 0 0 0"/>
+            <geometry>
+                <sphere radius="0.05"/>
+            </geometry>
+        </visual>
+        <collision name='front_caster_collision'>
+            <origin xyz="0.15 0 -0.05" rpy=" 0 0 0"/>
+            <geometry>
+                <sphere radius="0.05"/>
+            </geometry>
+            <surface>
+                <friction>
+                    <ode>
+                        <mu>0</mu>
+                        <mu2>0</mu2>
+                        <slip1>1.0</slip1>
+                        <slip2>1.0</slip2>
+                    </ode>
+                </friction>
+            </surface>
+        </collision>
+        <visual name='front_caster_visual'>
+            <origin xyz="0.15 0 -0.05" rpy=" 0 0 0"/>
+            <geometry>
+                <sphere radius="0.05"/>
+            </geometry>
+        </visual>
+    </link>
 </robot>
