Commit message: reverting udacity bot back to its original form

File: src/udacity_bot/urdf/udacity_bot.xacro (robot description, xacro)
@@ -1,453 +1,177 @@
 <?xml version='1.0'?>
 <robot name="udacity_bot" xmlns:xacro="http://www.ros.org/wiki/xacro">
-  <xacro:property name="chassissize"       value=".4 .4 .1" />
-  <xacro:property name="chassispose"       value="0 0 0.1 0 0 0" />
-  <xacro:property name="chassisorigin"     value="0.0 0.0 0.0" />
-  <xacro:property name="wheelradius"       value="0.1" />
-  <xacro:property name="wheellength"       value="0.05" />
-  <xacro:property name="leftwheelorigin"   value="0.0  0.0 0.0" />
-  <xacro:property name="rightwheelorigin"  value="0.0  0.0 0.0" />
-  <xacro:property name="leftwheelhinge"    value="0 0.23 0" />
-  <xacro:property name="rightwheelhinge"   value="0 -0.23 0" />
-  <xacro:property name="casterradius"      value="0.05" />
-  <xacro:property name="frontcasterorigin" value="-0.15 0 -0.05" />
-  <xacro:property name="backcasterorigin"  value=" 0.15 0 -0.05" />
-  <xacro:property name="camerasize"        value="0.05 0.05 0.05" />
-	<xacro:property name="cameraorigin"      value="0.0 0.0 0.0" />
-	<xacro:property name="hokuyoorigin"      value="0.0 0.0 0.0" />
-  <xacro:property name="torsolink"         value="0.0 0.0 0.1" />
-  <xacro:property name="torsoradius"       value="0.1" />
-  <xacro:property name="torsolength"       value="0.2" />
-  <xacro:property name="torsoorigin"       value="0.0 0.0 0.0" />
-  <xacro:property name="polelength"        value="0.2" />
-  <xacro:property name="width"             value="0.15" />
-  <xacro:include filename="$(find udacity_bot)/urdf/udacity_bot.gazebo" />
-	<!-- Import Rviz colors -->
-  <xacro:include filename="$(find udacity_bot)/urdf/materials.xacro" />
-  <link name="robot_footprint"></link>
-  <joint name="robot_footprint_joint" type="fixed">
-    <origin xyz="0 0 0" rpy="0 0 0" />
-    <parent link="robot_footprint"/>
-    <child link="chassis" />
-  </joint>
-  <link name='chassis'>
-    <pose>${chassispose}</pose>
-    <inertial>
-      <mass value="15.0"/>
-      <origin xyz="0.0 0 0" rpy=" 0 0 0"/>
-      <inertia
-          ixx="0.1" ixy="0" ixz="0"
-          iyy="0.1" iyz="0"
-          izz="0.1"
-      />
-    </inertial>
-    <collision name='collision'>
-      <origin xyz="0 0 0" rpy=" 0 0 0"/>
-      <geometry>
-        <box size="${chassissize}"/>
-      </geometry>
-    </collision>
-    <visual name='chassis_visual'>
-      <origin xyz="0 0 0" rpy=" 0 0 0"/>
-      <geometry>
-        <box size="${chassissize}"/>
-      </geometry>
-      <material name="red"/>
-   </visual>
-    <collision name='back_caster_collision'>
-      <origin xyz="${backcasterorigin}" rpy=" 0 0 0"/>
-      <geometry>
-        <sphere radius="${casterradius}"/>
-      </geometry>
-      <surface>
-        <friction>
-          <ode>
-            <mu>0</mu>
-            <mu2>0</mu2>
-            <slip1>1.0</slip1>
-            <slip2>1.0</slip2>
-          </ode>
-        </friction>
-      </surface>
-    </collision>
-    <visual name='back_caster_visual'>
-      <origin xyz="${backcasterorigin}" rpy=" 0 0 0"/>
-      <geometry>
-        <sphere radius="0.05"/>
-      </geometry>
-    </visual>
-    <collision name='front_caster_collision'>
-      <origin xyz="${frontcasterorigin}" rpy=" 0 0 0"/>
-      <geometry>
-        <sphere radius="${casterradius}"/>
-      </geometry>
-      <surface>
-        <friction>
-          <ode>
-            <mu>0</mu>
-            <mu2>0</mu2>
-            <slip1>1.0</slip1>
-            <slip2>1.0</slip2>
-          </ode>
-        </friction>
-      </surface>
-    </collision>
-    <visual name='front_caster_visual'>
-      <origin xyz="${frontcasterorigin}" rpy=" 0 0 0"/>
-      <geometry>
-        <sphere radius="${casterradius}"/>
-      </geometry>
-    </visual>
-  </link>
-	<link name="torso">
-	 <collision name='torsocollision'>
-      <origin xyz="${torsoorigin}" rpy=" 0 0 0"/>
-      <geometry>
-          <cylinder radius="${torsoradius}" length="${torsolength}"/>
-      </geometry>
-    </collision>
-		 <inertial>
-      <mass value="5.0"/>
-      <origin xyz="${torsoorigin}" rpy=" 0 0 0"/>
-      <inertia
-          ixx="0.1" ixy="0" ixz="0"
-          iyy="0.1" iyz="0"
-          izz="0.1"
-      />
-    </inertial>
-    <visual name='torso_visual'>
-      <origin xyz="${torsoorigin}" rpy=" 0 0 0"/>
-      <geometry>
-          <cylinder radius="${torsoradius}" length="${torsolength}"/>
-      </geometry>
-      <material name="black"/>
-   </visual>
-	</link>
-	<joint type="continuous" name="torsolink">
-    <origin xyz="${torsolink}" rpy="0 0 0"/>
-    <child link="torso"/>
-    <parent link="chassis"/>
-    <axis xyz="0 0 1" rpy="0 0 0"/>
-    <limit effort="10000" velocity="1000"/>
-    <joint_properties damping="1.0" friction="1.0"/>
-  </joint>
-  <link name="left_wheel">
-    <collision name='left_wheel_collision'>
-      <origin xyz="${leftwheelorigin}" rpy=" 0.0 1.5707 1.5707"/>
-      <geometry>
-        <cylinder radius="${wheelradius}" length="${wheellength}"/>
-      </geometry>
-      <surface>
-        <friction>
-          <ode>
-            <mu>0</mu>
-            <mu2>0</mu2>
-            <slip1>1.0</slip1>
-            <slip2>1.0</slip2>
-          </ode>
-        </friction>
-      </surface>
-    </collision>
-    <inertial>
-      <mass value="5.0"/>
-      <origin xyz="${leftwheelorigin}" rpy=" 0 0 0"/>
-      <inertia
-          ixx="0.1" ixy="0" ixz="0"
-          iyy="0.1" iyz="0"
-          izz="0.1"
-      />
-    </inertial>
-    <visual name='left_wheel_visual'>
-     <origin xyz="${leftwheelorigin}" rpy=" 0.0 1.5707 1.5707"/>
-      <geometry>
-        <cylinder radius="${wheelradius}" length="${wheellength}"/>
-      </geometry>
-      <material name="black"/>
-    </visual>
-  </link>
-  <joint type="continuous" name="left_wheel_hinge">
-    <origin xyz="${leftwheelhinge}" rpy="0 0 0"/>
-    <child link="left_wheel"/>
-    <parent link="chassis"/>
-    <axis xyz="0 1 0" rpy="0 0 0"/>
-    <limit effort="10000" velocity="1000"/>
-    <joint_properties damping="1.0" friction="1.0"/>
-  </joint>
-  <link name="right_wheel">
-    <collision name='right_wheel_collision'>
-      <origin xyz="${rightwheelorigin}" rpy=" 0.0 1.5707 1.5707"/>
-      <geometry>
-        <cylinder radius="${wheelradius}" length="${wheellength}"/>
-      </geometry>
-      <surface>
-        <friction>
-          <ode>
-            <mu>0</mu>
-            <mu2>0</mu2>
-            <slip1>1.0</slip1>
-            <slip2>1.0</slip2>
-          </ode>
-        </friction>
-      </surface>
-    </collision>
-    <inertial>
-      <mass value="5.0"/>
-      <origin xyz="0.0 0.0 0.0" rpy=" 0.0 0.0 0.0"/>
-      <inertia
-          ixx="0.1" ixy="0" ixz="0"
-          iyy="0.1" iyz="0"
-          izz="0.1"
-      />
-    </inertial>
-    <visual name='right_wheel_visual'>
-      <origin xyz="${rightwheelorigin}" rpy=" 0.0 1.5707 1.5707"/>
-      <geometry>
-        <cylinder radius="${wheelradius}" length="${wheellength}"/>
-      </geometry>
-       <material name="black"/>
-   </visual>
-  </link>
-  <joint type="continuous" name="right_wheel_hinge">
-    <origin xyz="${rightwheelhinge}" rpy="0 0 0"/>
-    <child link="right_wheel"/>
-    <parent link="chassis"/>
-    <axis xyz="0 1 0" rpy="0 0 0"/>
-    <limit effort="10000" velocity="1000"/>
-    <joint_properties damping="1.0" friction="1.0"/>
-  </joint>
-  <link name="camera">
-    <collision name='camera_collision'>
-      <origin xyz="${cameraorigin}" rpy=" 0.0 0.0 0.0"/>
-      <geometry>
-        <box size="${camerasize}"/>
-      </geometry>
-      <surface>
-        <friction>
-          <ode>
-            <mu>0</mu>
-            <mu2>0</mu2>
-            <slip1>1.0</slip1>
-            <slip2>1.0</slip2>
-          </ode>
-        </friction>
-      </surface>
-    </collision>
-    <inertial>
-      <mass value="0.1"/>
-      <origin xyz="0.0 0.0 0.0" rpy=" 0.0 0.0 0.0"/>
-      <inertia
-          ixx="1e-6" ixy="0" ixz="0"
-          iyy="1e-6" iyz="0"
-          izz="1e-6"
-      />
-    </inertial>
-    <visual name='camera_visual'>
-      <origin xyz="${cameraorigin}" rpy=" 0.0 0.0 0.0"/>
-      <geometry>
-        <box size="${camerasize}"/>
-      </geometry>
-      <material name="orange"/>
-    </visual>
-  </link>
-  <joint type="continuous" name="camera_joint">
-    <origin xyz="0.2 0.0 0.0" rpy="0 0 0"/>
-    <child link="camera"/>
-    <parent link="chassis"/>
-    <axis xyz="0 1 0" rpy="0 0 0"/>
-    <limit effort="10000" velocity="1000"/>
-    <joint_properties damping="1.0" friction="1.0"/>
-  </joint>
-  <link name="hokuyo">
-    <collision name='hokuyo_collision'>
-      <origin xyz="${hokuyoorigin}" rpy=" 0.0 0.0 0.0"/>
-      <geometry>
-        <box size="0.1 0.1 0.1"/>
-      </geometry>
-      <surface>
-        <friction>
-          <ode>
-            <mu>0</mu>
-            <mu2>0</mu2>
-            <slip1>1.0</slip1>
-            <slip2>1.0</slip2>
-          </ode>
-        </friction>
-      </surface>
-    </collision>
-    <inertial>
-      <mass value="0.1"/>
-      <origin xyz="${hokuyoorigin}" rpy=" 0.0 0.0 0.0"/>
-      <inertia
-          ixx="1e-6" ixy="0" ixz="0"
-          iyy="1e-6" iyz="0"
-          izz="1e-6"
-      />
-    </inertial>
-    <visual name='hokuyo_visual'>
-      <origin xyz="${hokuyoorigin}" rpy=" 0.0 0.0 0.0"/>
-      <geometry>
-        <mesh filename="package://udacity_bot/meshes/hokuyo.dae"/>
-      </geometry>
-   </visual>
-  </link>
-  <joint type="continuous" name="hokuyo_joint">
-    <origin xyz="0.0 0.0 0.225" rpy="0 0 0"/>
-    <child link="hokuyo"/>
-    <parent link="chassis"/>
-    <axis xyz="0 1 0" rpy="0 0 0"/>
-    <limit effort="10000" velocity="1000"/>
-    <joint_properties damping="1.0" friction="1.0"/>
-  </joint>
-  <xacro:macro name="default_inertial" params="mass">
-    <inertial>
-      <mass value="${mass}" />
-      <inertia ixx="1.0" ixy="0.0" ixz="0.0" iyy="1.0" iyz="0.0" izz="1.0" />
-    </inertial>
-  </xacro:macro>
-	<!-- Gripper1 (left) -->
-  <joint name="gripper_extension1" type="prismatic">
-		<origin xyz="0.0 0.09 0.08" rpy="0 0 0"/>
-    <parent link="torso"/>
-    <child link="gripper_pole1"/>
-    <limit effort="1000.0" lower="-${width*2-.02}" upper="0" velocity="0.5"/>
-    <origin rpy="0 0 0" xyz="0 0 0.15"/>
-    <limit effort="30" velocity="0.2"/>
-    <dynamics damping="1.0" friction="1.0"/>
-  </joint>
-	<link name="gripper_pole1">
-    <visual>
-      <geometry>
-        <cylinder length="${polelength}" radius="0.01"/>
-      </geometry>
-      <origin xyz="${polelength/2} 0 0" rpy="0 ${pi/2} 0 "/>
-      <material name="grey"/>
-    </visual>
-    <collision>
-      <geometry>
-        <cylinder length="${polelength}" radius="0.01"/>
-      </geometry>
-      <origin xyz="${polelength/2} 0 0" rpy="0 0 0 "/>
-    </collision>
-    <xacro:default_inertial mass="0.05"/>
-  </link>
-  <xacro:macro name="gripper1" params="prefix reflect">
-    <joint name="${prefix}_gripper_joint1" type="revolute">
-      <axis xyz="0 0 ${reflect}"/>
-      <limit effort="1000.0" lower="0.0" upper="0.548" velocity="0.5"/>
-      <origin rpy="0 0 0" xyz="${polelength} ${reflect*0.01} 0"/>
-      <parent link="gripper_pole1"/>
-      <child link="${prefix}_gripper1"/>
-      <limit effort="30" velocity="1.0"/>
-      <dynamics damping="0.0" friction="0.0"/>
+    <xacro:include filename="$(find udacity_bot)/urdf/udacity_bot.gazebo" />
+    <link name="robot_footprint"></link>
+    <joint name="robot_footprint_joint" type="fixed">
+        <origin xyz="0 0 0" rpy="0 0 0"/>
+        <parent link="robot_footprint"/>
+        <child link="chassis"/>
     </joint>
-		<link name="${prefix}_gripper1">
-      <visual>
-        <origin rpy="${(reflect-1)/2*pi} 0 0" xyz="0 0 0"/>
-        <geometry>
-          <mesh filename="package://udacity_bot/meshes/l_finger.dae"/>
-        </geometry>
-      </visual>
-      <collision>
-        <geometry>
-          <mesh filename="package://udacity_bot/meshes/l_finger.dae"/>
-        </geometry>
-        <origin rpy="${(reflect-1)/2*pi} 0 0" xyz="0 0 0"/>
-      </collision>
-      <xacro:default_inertial mass="0.05"/>
+    <link name='left_wheel'>
+        <inertial>
+            <mass value="5.0"/>
+            <origin xyz="0.0 0 0" rpy=" 0 1.5707 1.5707"/>
+            <inertia ixx="0.1" ixy="0" ixz="0" iyy="0.1" iyz="0" izz="0.1"/>
+        </inertial>
+        <collision name='collision'>
+            <origin xyz="0.0 0 0" rpy=" 0 1.5707 1.5707"/>
+            <geometry>
+                <cylinder length="0.05" radius="0.1"/>
+            </geometry>
+        </collision>
+        <visual name='wheel_visual'>
+            <origin xyz="0.0 0 0" rpy=" 0 1.5707 1.5707"/>
+            <geometry>
+                <cylinder length="0.05" radius="0.1"/>
+            </geometry>
+        </visual>
     </link>
-    <joint name="${prefix}_tip_joint1" type="fixed">
-      <parent link="${prefix}_gripper1"/>
-      <child link="${prefix}_tip1"/>
+    <joint type="continuous" name="left_wheel_hinge">
+        <origin xyz="0 0.15 0" rpy="0 0 0"/>
+        <child link="left_wheel"/>
+        <parent link="chassis"/>
+        <axis xyz="0 1 0" rpy="0 0 0"/>
+        <limit effort="10000" velocity="1000"/>
+        <joint_properties damping="1.0" friction="1.0"/>
     </joint>
-    <link name="${prefix}_tip1">
-      <visual>
-        <origin rpy="${(reflect-1)/2*pi} 0 0" xyz="0.09137 0.00495 0"/>
-        <geometry>
-          <mesh filename="package://udacity_bot/meshes/l_finger_tip.dae"/>
-        </geometry>
-      </visual>
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