Commit message: first iteration of martin_bot

File: src/martin_bot/urdf/martin_bot.xacro (robot description, xacro)
@@ -1,4 +1,47 @@
 <?xml version='1.0'?>
 <robot name="martin_bot" xmlns:xacro="http://www.ros.org/wiki/xacro">
+  <xacro:property name="chassissize"       value=".4 .2 .1" />
+  <xacro:property name="chassispose"       value="0 0 0.1 0 0 0" />
+  <xacro:property name="chassisorigin"     value="0.0 0.0 0.06" />
+  <xacro:property name="wheelradius"       value="0.1" />
+  <xacro:property name="wheellength"       value="0.05" />
+  <xacro:property name="leftwheelorigin"   value="0.0  0.0 0.0" />
+  <xacro:property name="rightwheelorigin"  value="0.0  0.0 0.0" />
+  <xacro:property name="leftwheelhinge"    value="0 0.15 0" />
+  <xacro:property name="rightwheelhinge"   value="0 -0.15 0" />
+  <xacro:property name="casterradius"      value="0.05" />
+  <xacro:property name="frontcasterorigin" value="-0.15 0 -0.05" />
+  <xacro:property name="backcasterorigin"  value=" 0.15 0 -0.05" />
+  <xacro:property name="camerasize"        value="0.05 0.05 0.05" />
+  <xacro:property name="towerradius"       value="0.1" />
+  <xacro:property name="towerlength"       value="0.3" />
+  <xacro:property name="towerorigin"       value="0.0 0.0 0.06" />
+  <xacro:property name="polelen"           value="0.2" />
+  <xacro:property name="width"             value="0.2" />
+  <material name="blue">
+    <color rgba="0.12 0.56 1.0 1"/>
+  </material>
+  <material name="turquoise">
+    <color rgba="0.25 0.88 0.82 1"/>
+  </material>
+  <material name="yellow">
+    <color rgba="1.0 0.84 0 1"/>
+  </material>
+  <material name="purple">
+    <color rgba="0.8 0 0.8 1"/>
+  </material>
+  <material name="green">
+    <color rgba="013 0.55 0.13 1"/>
+  </material>
+  <material name="red">
+    <color rgba="0.86 0.08 0.24 1"/>
+  </material>
+  <material name="black">
+    <color rgba="0 0 0 1"/>
+  </material>
+  <material name="white">
+    <color rgba="1 1 1 1"/>
+  </material>
+  <xacro:include filename="$(find martin_bot)/urdf/martin_bot.gazebo" />
   <link name="robot_footprint"></link>
   <joint name="robot_footprint_joint" type="fixed">
@@ -8,5 +51,5 @@
   </joint>
   <link name='chassis'>
-    <pose>0 0 0.1 0 0 0</pose>
+    <pose>${chassispose}</pose>
     <inertial>
       <mass value="15.0"/>
@@ -21,5 +64,5 @@
       <origin xyz="0 0 0" rpy=" 0 0 0"/>
       <geometry>
-        <box size=".4 .2 .1"/>
+        <box size="${chassissize}"/>
       </geometry>
     </collision>
@@ -27,33 +70,47 @@
       <origin xyz="0 0 0" rpy=" 0 0 0"/>
       <geometry>
-        <box size=".4 .2 .1"/>
-      </geometry>
-    </visual>
+        <box size="${chassissize}"/>
+      </geometry>
+      <material name="blue"/>
+   </visual>
+    <collision name='towercollision'>
+      <origin xyz="${towerorigin}" rpy=" 0 0 0"/>
+      <geometry>
+          <cylinder radius="${towerradius}" length="${towerlength}"/>
+      </geometry>
+    </collision>
+    <visual name='tower_visual'>
+      <origin xyz="${towerorigin}" rpy=" 0 0 0"/>
+      <geometry>
+          <cylinder radius="${towerradius}" length="${towerlength}"/>
+      </geometry>
+      <material name="green"/>
+   </visual>
     <collision name='back_caster_collision'>
-      <origin xyz="-0.15 0 -0.05" rpy=" 0 0 0"/>
+      <origin xyz="${backcasterorigin}" rpy=" 0 0 0"/>
+      <geometry>
+        <sphere radius="${casterradius}"/>
+      </geometry>
+      <surface>
+        <friction>
+          <ode>
+            <mu>0</mu>
+            <mu2>0</mu2>
+            <slip1>1.0</slip1>
+            <slip2>1.0</slip2>
+          </ode>
+        </friction>
+      </surface>
+    </collision>
+    <visual name='back_caster_visual'>
+      <origin xyz="${backcasterorigin}" rpy=" 0 0 0"/>
       <geometry>
         <sphere radius="0.05"/>
       </geometry>
-      <surface>
-        <friction>
-          <ode>
-            <mu>0</mu>
-            <mu2>0</mu2>
-            <slip1>1.0</slip1>
-            <slip2>1.0</slip2>
-          </ode>
-        </friction>
-      </surface>
-    </collision>
-    <visual name='back_caster_visual'>
-      <origin xyz="-0.15 0 -0.05" rpy=" 0 0 0"/>
-      <geometry>
-        <sphere radius="0.05"/>
-      </geometry>
     </visual>
     <collision name='front_caster_collision'>
-      <origin xyz="0.15 0 -0.05" rpy=" 0 0 0"/>
-      <geometry>
-        <sphere radius="0.05"/>
+      <origin xyz="${frontcasterorigin}" rpy=" 0 0 0"/>
+      <geometry>
+        <sphere radius="${casterradius}"/>
       </geometry>
       <surface>
@@ -69,9 +126,253 @@
     </collision>
     <visual name='front_caster_visual'>
-      <origin xyz="0.15 0 -0.05" rpy=" 0 0 0"/>
-      <geometry>
-        <sphere radius="0.05"/>
-      </geometry>
-    </visual>
-  </link>
+      <origin xyz="${frontcasterorigin}" rpy=" 0 0 0"/>
+      <geometry>
+        <sphere radius="${casterradius}"/>
+      </geometry>
+    </visual>
+  </link>
+  <link name="left_wheel">
+    <collision name='left_wheel_collision'>
+      <origin xyz="${leftwheelorigin}" rpy=" 0.0 1.5707 1.5707"/>
+      <geometry>
+        <cylinder radius="${wheelradius}" length="${wheellength}"/>
+      </geometry>
+      <surface>
+        <friction>
+          <ode>
+            <mu>0</mu>
+            <mu2>0</mu2>
+            <slip1>1.0</slip1>
+            <slip2>1.0</slip2>
+          </ode>
+        </friction>
+      </surface>
+    </collision>
+    <inertial>
+      <mass value="5.0"/>
+      <origin xyz="${leftwheelorigin}" rpy=" 0 0 0"/>
+      <inertia
+          ixx="0.1" ixy="0" ixz="0"
+          iyy="0.1" iyz="0"
+          izz="0.1"
+      />
+    </inertial>
+    <visual name='left_wheel_visual'>
+     <origin xyz="${leftwheelorigin}" rpy=" 0.0 1.5707 1.5707"/>
+      <geometry>
+        <cylinder radius="${wheelradius}" length="${wheellength}"/>
+      </geometry>
+      <material name="yellow"/>
+    </visual>
+  </link>
+  <joint type="continuous" name="left_wheel_hinge">
+    <origin xyz="${leftwheelhinge}" rpy="0 0 0"/>
+    <child link="left_wheel"/>
+    <parent link="chassis"/>
+    <axis xyz="0 1 0" rpy="0 0 0"/>
+    <limit effort="10000" velocity="1000"/>
+    <joint_properties damping="1.0" friction="1.0"/>
+  </joint>
+  <link name="right_wheel">
+    <collision name='right_wheel_collision'>
+      <origin xyz="${rightwheelorigin}" rpy=" 0.0 1.5707 1.5707"/>
+      <geometry>
+        <cylinder radius="${wheelradius}" length="${wheellength}"/>
+      </geometry>
+      <surface>
+        <friction>
+          <ode>
+            <mu>0</mu>
+            <mu2>0</mu2>
+            <slip1>1.0</slip1>
+            <slip2>1.0</slip2>
+          </ode>
+        </friction>
+      </surface>
+    </collision>
+    <inertial>
+      <mass value="5.0"/>
+      <origin xyz="0.0 0.0 0.0" rpy=" 0.0 0.0 0.0"/>
+      <inertia
+          ixx="0.1" ixy="0" ixz="0"
+          iyy="0.1" iyz="0"
+          izz="0.1"
+      />
+    </inertial>
+    <visual name='right_wheel_visual'>
+      <origin xyz="${rightwheelorigin}" rpy=" 0.0 1.5707 1.5707"/>
+      <geometry>
+        <cylinder radius="${wheelradius}" length="${wheellength}"/>
+      </geometry>
+       <material name="yellow"/>
+   </visual>
+  </link>
+  <joint type="continuous" name="right_wheel_hinge">
+    <origin xyz="${rightwheelhinge}" rpy="0 0 0"/>
+    <child link="right_wheel"/>
+    <parent link="chassis"/>
+    <axis xyz="0 1 0" rpy="0 0 0"/>
+    <limit effort="10000" velocity="1000"/>
+    <joint_properties damping="1.0" friction="1.0"/>
+  </joint>
+  <link name="camera">
+    <collision name='camera_collision'>
+      <origin xyz="0.0 0.0 0.0" rpy=" 0.0 0.0 0.0"/>
+      <geometry>
+        <box size="${camerasize}"/>
+      </geometry>
+      <surface>
+        <friction>
+          <ode>
+            <mu>0</mu>
+            <mu2>0</mu2>
+            <slip1>1.0</slip1>
+            <slip2>1.0</slip2>
+          </ode>
+        </friction>
+      </surface>
+    </collision>
+    <inertial>
+      <mass value="0.1"/>
+      <origin xyz="0.0 0.0 0.0" rpy=" 0.0 0.0 0.0"/>
+      <inertia
+          ixx="1e-6" ixy="0" ixz="0"
+          iyy="1e-6" iyz="0"
+          izz="1e-6"
+      />
+    </inertial>
+    <visual name='camera_visual'>
+      <origin xyz="0.0 0.0 0.0" rpy=" 0.0 0.0 0.0"/>
+      <geometry>
+        <box size="${camerasize}"/>
+      </geometry>
+      <material name="turquoise"/>
+    </visual>
+  </link>
+  <joint type="continuous" name="camera_joint">
+    <origin xyz="0.2 0.0 0.0" rpy="0 0 0"/>
+    <child link="camera"/>
+    <parent link="chassis"/>
+    <axis xyz="0 1 0" rpy="0 0 0"/>
+    <limit effort="10000" velocity="1000"/>
+    <joint_properties damping="1.0" friction="1.0"/>
+  </joint>
+  <link name="hokuyo">
+    <collision name='hokuyo_collision'>
+      <origin xyz="0.0 0.0 0.0" rpy=" 0.0 0.0 0.0"/>
+      <geometry>
+        <box size="0.1 0.1 0.1"/>
+      </geometry>
+      <surface>
+        <friction>
+          <ode>
+            <mu>0</mu>
+            <mu2>0</mu2>
+            <slip1>1.0</slip1>
+            <slip2>1.0</slip2>
+          </ode>
+        </friction>
+      </surface>
+    </collision>
+    <inertial>
+      <mass value="0.1"/>
+      <origin xyz="0.0 0.0 0.0" rpy=" 0.0 0.0 0.0"/>
+      <inertia
+          ixx="1e-6" ixy="0" ixz="0"
+          iyy="1e-6" iyz="0"
+          izz="1e-6"
+      />
+    </inertial>
+    <visual name='hokuyo_visual'>
+      <origin xyz="0.0 0.0 0.0" rpy=" 0.0 0.0 0.0"/>
+      <geometry>
+        <mesh filename="package://martin_bot/meshes/hokuyo.dae"/>
+      </geometry>
+   </visual>
+  </link>
+  <joint type="continuous" name="hokuyo_joint">
+    <origin xyz="0.0 0.0 0.225" rpy="0 0 0"/>
+    <child link="hokuyo"/>
+    <parent link="chassis"/>
+    <axis xyz="0 1 0" rpy="0 0 0"/>
+    <limit effort="10000" velocity="1000"/>
+    <joint_properties damping="1.0" friction="1.0"/>
+  </joint>
+  <xacro:macro name="default_inertial" params="mass">
+    <inertial>
+      <mass value="${mass}" />
+      <inertia ixx="1.0" ixy="0.0" ixz="0.0" iyy="1.0" iyz="0.0" izz="1.0" />
+    </inertial>
+  </xacro:macro>
+  <joint name="gripper_extension" type="prismatic">
+    <parent link="robot_footprint"/>
+    <child link="gripper_pole"/>
+    <limit effort="1000.0" lower="-${width*2-.02}" upper="0" velocity="0.5"/>
+    <origin rpy="0 0 0" xyz="0 0 0.15"/>
+    <limit effort="30" velocity="0.2"/>
+    <dynamics damping="1.0" friction="1.0"/>
+  </joint>
+  <link name="gripper_pole">
+    <visual>
+      <geometry>
+        <cylinder length="${polelen}" radius="0.01"/>
+      </geometry>
+      <origin xyz="${polelen/2} 0 0" rpy="0 ${pi/2} 0 "/>
+      <material name="green"/>
+    </visual>
+    <collision>
+      <geometry>
+        <cylinder length="${polelen}" radius="0.01"/>
+      </geometry>
+      <origin xyz="${polelen/2} 0 0" rpy="0 0 0 "/>
+    </collision>
+    <xacro:default_inertial mass="0.05"/>
+  </link>
+  <xacro:macro name="gripper" params="prefix reflect">
+    <joint name="${prefix}_gripper_joint" type="revolute">
+      <axis xyz="0 0 ${reflect}"/>
+      <limit effort="1000.0" lower="0.0" upper="0.548" velocity="0.5"/>
+      <origin rpy="0 0 0" xyz="${polelen} ${reflect*0.01} 0"/>
+      <parent link="gripper_pole"/>
+      <child link="${prefix}_gripper"/>
+      <limit effort="30" velocity="1.0"/>
+      <dynamics damping="0.0" friction="0.0"/>
+    </joint>
+    <link name="${prefix}_gripper">
+      <visual>
+        <origin rpy="${(reflect-1)/2*pi} 0 0" xyz="0 0 0"/>
+        <geometry>
+          <mesh filename="package://martin_bot/meshes/l_finger.dae"/>
+        </geometry>
+      </visual>
+      <collision>
+        <geometry>
+          <mesh filename="package://martin_bot/meshes/l_finger.dae"/>
+        </geometry>
+        <origin rpy="${(reflect-1)/2*pi} 0 0" xyz="0 0 0"/>
+      </collision>
+      <xacro:default_inertial mass="0.05"/>
+    </link>
+    <joint name="${prefix}_tip_joint" type="fixed">
+      <parent link="${prefix}_gripper"/>
+      <child link="${prefix}_tip"/>
+    </joint>
+    <link name="${prefix}_tip">
+      <visual>
+        <origin rpy="${(reflect-1)/2*pi} 0 0" xyz="0.09137 0.00495 0"/>
+        <geometry>
+          <mesh filename="package://martin_bot/meshes/l_finger_tip.dae"/>
+        </geometry>
+      </visual>
+      <collision>
+        <geometry>
+          <mesh filename="package://martin_bot/meshes/l_finger_tip.dae"/>
+        </geometry>
+        <origin rpy="${(reflect-1)/2*pi} 0 0" xyz="0.09137 0.00495 0"/>
+      </collision>
+      <xacro:default_inertial mass="0.05"/>
+    </link>
+  </xacro:macro>
+  <xacro:gripper prefix="left" reflect="1" />
+  <xacro:gripper prefix="right" reflect="-1" />
 </robot>

Commit message: materials file and macros

File: src/martin_bot/urdf/martin_bot.xacro (robot description, xacro)
@@ -1,5 +1,5 @@
 <?xml version='1.0'?>
 <robot name="martin_bot" xmlns:xacro="http://www.ros.org/wiki/xacro">
-  <xacro:property name="chassissize"       value=".4 .2 .1" />
+  <xacro:property name="chassissize"       value=".4 .4 .1" />
   <xacro:property name="chassispose"       value="0 0 0.1 0 0 0" />
   <xacro:property name="chassisorigin"     value="0.0 0.0 0.06" />
@@ -8,40 +8,20 @@
   <xacro:property name="leftwheelorigin"   value="0.0  0.0 0.0" />
   <xacro:property name="rightwheelorigin"  value="0.0  0.0 0.0" />
-  <xacro:property name="leftwheelhinge"    value="0 0.15 0" />
-  <xacro:property name="rightwheelhinge"   value="0 -0.15 0" />
+  <xacro:property name="leftwheelhinge"    value="0 0.25 0" />
+  <xacro:property name="rightwheelhinge"   value="0 -0.25 0" />
   <xacro:property name="casterradius"      value="0.05" />
   <xacro:property name="frontcasterorigin" value="-0.15 0 -0.05" />
   <xacro:property name="backcasterorigin"  value=" 0.15 0 -0.05" />
   <xacro:property name="camerasize"        value="0.05 0.05 0.05" />
+	<xacro:property name="cameraorigin"      value="0.0 0.0 0.0" />
+	<xacro:property name="hokuyoorigin"      value="0.0 0.0 0.0" />
   <xacro:property name="towerradius"       value="0.1" />
-  <xacro:property name="towerlength"       value="0.3" />
-  <xacro:property name="towerorigin"       value="0.0 0.0 0.06" />
-  <xacro:property name="polelen"           value="0.2" />
+  <xacro:property name="towerlength"       value="0.2" />
+  <xacro:property name="towerorigin"       value="0.0 0.0 0.1" />
+  <xacro:property name="polelen"           value="0.3" />
   <xacro:property name="width"             value="0.2" />
-  <material name="blue">
-    <color rgba="0.12 0.56 1.0 1"/>
-  </material>
-  <material name="turquoise">
-    <color rgba="0.25 0.88 0.82 1"/>
-  </material>
-  <material name="yellow">
-    <color rgba="1.0 0.84 0 1"/>
-  </material>
-  <material name="purple">
-    <color rgba="0.8 0 0.8 1"/>
-  </material>
-  <material name="green">
-    <color rgba="013 0.55 0.13 1"/>
-  </material>
-  <material name="red">
-    <color rgba="0.86 0.08 0.24 1"/>
-  </material>
-  <material name="black">
-    <color rgba="0 0 0 1"/>
-  </material>
-  <material name="white">
-    <color rgba="1 1 1 1"/>
-  </material>
   <xacro:include filename="$(find martin_bot)/urdf/martin_bot.gazebo" />
+	<!-- Import Rviz colors -->
+  <xacro:include filename="$(find martin_bot)/urdf/materials.xacro" />
   <link name="robot_footprint"></link>
   <joint name="robot_footprint_joint" type="fixed">
@@ -72,5 +52,5 @@
         <box size="${chassissize}"/>
       </geometry>
-      <material name="blue"/>
+      <material name="red"/>
    </visual>
     <collision name='towercollision'>
@@ -163,5 +143,5 @@
         <cylinder radius="${wheelradius}" length="${wheellength}"/>
       </geometry>
-      <material name="yellow"/>
+      <material name="black"/>
     </visual>
   </link>
@@ -205,5 +185,5 @@
         <cylinder radius="${wheelradius}" length="${wheellength}"/>
       </geometry>
-       <material name="yellow"/>
+       <material name="black"/>
    </visual>
   </link>
@@ -218,5 +198,5 @@
   <link name="camera">
     <collision name='camera_collision'>
-      <origin xyz="0.0 0.0 0.0" rpy=" 0.0 0.0 0.0"/>
+      <origin xyz="${cameraorigin}" rpy=" 0.0 0.0 0.0"/>
       <geometry>
         <box size="${camerasize}"/>
@@ -243,5 +223,5 @@
     </inertial>
     <visual name='camera_visual'>
-      <origin xyz="0.0 0.0 0.0" rpy=" 0.0 0.0 0.0"/>
+      <origin xyz="${cameraorigin}" rpy=" 0.0 0.0 0.0"/>
       <geometry>
         <box size="${camerasize}"/>
@@ -260,5 +240,5 @@
   <link name="hokuyo">
     <collision name='hokuyo_collision'>
-      <origin xyz="0.0 0.0 0.0" rpy=" 0.0 0.0 0.0"/>
+      <origin xyz="${hokuyoorigin}" rpy=" 0.0 0.0 0.0"/>
       <geometry>
         <box size="0.1 0.1 0.1"/>
@@ -277,5 +257,5 @@
     <inertial>
       <mass value="0.1"/>
-      <origin xyz="0.0 0.0 0.0" rpy=" 0.0 0.0 0.0"/>
+      <origin xyz="${hokuyoorigin}" rpy=" 0.0 0.0 0.0"/>
       <inertia
           ixx="1e-6" ixy="0" ixz="0"
@@ -285,5 +265,5 @@
     </inertial>
     <visual name='hokuyo_visual'>
-      <origin xyz="0.0 0.0 0.0" rpy=" 0.0 0.0 0.0"/>
+      <origin xyz="${hokuyoorigin}" rpy=" 0.0 0.0 0.0"/>
       <geometry>
         <mesh filename="package://martin_bot/meshes/hokuyo.dae"/>

Commit message: materials

File: src/martin_bot/urdf/martin_bot.xacro (robot description, xacro)
@@ -16,8 +16,8 @@
 	<xacro:property name="cameraorigin"      value="0.0 0.0 0.0" />
 	<xacro:property name="hokuyoorigin"      value="0.0 0.0 0.0" />
-  <xacro:property name="towerradius"       value="0.1" />
-  <xacro:property name="towerlength"       value="0.2" />
-  <xacro:property name="towerorigin"       value="0.0 0.0 0.1" />
-  <xacro:property name="polelen"           value="0.3" />
+  <xacro:property name="torsoradius"       value="0.1" />
+  <xacro:property name="torsolength"       value="0.2" />
+  <xacro:property name="torsoorigin"       value="0.0 0.0 0.1" />
+  <xacro:property name="polelength"        value="0.3" />
   <xacro:property name="width"             value="0.2" />
   <xacro:include filename="$(find martin_bot)/urdf/martin_bot.gazebo" />
@@ -54,14 +54,14 @@
       <material name="red"/>
    </visual>
-    <collision name='towercollision'>
-      <origin xyz="${towerorigin}" rpy=" 0 0 0"/>
-      <geometry>
-          <cylinder radius="${towerradius}" length="${towerlength}"/>
-      </geometry>
-    </collision>
-    <visual name='tower_visual'>
-      <origin xyz="${towerorigin}" rpy=" 0 0 0"/>
-      <geometry>
-          <cylinder radius="${towerradius}" length="${towerlength}"/>
+    <collision name='torsocollision'>
+      <origin xyz="${torsoorigin}" rpy=" 0 0 0"/>
+      <geometry>
+          <cylinder radius="${torsoradius}" length="${torsolength}"/>
+      </geometry>
+    </collision>
+    <visual name='torso_visual'>
+      <origin xyz="${torsoorigin}" rpy=" 0 0 0"/>
+      <geometry>
+          <cylinder radius="${torsoradius}" length="${torsolength}"/>
       </geometry>
       <material name="green"/>
@@ -227,5 +227,5 @@
         <box size="${camerasize}"/>
       </geometry>
-      <material name="turquoise"/>
+      <material name="orange"/>
     </visual>
   </link>
@@ -296,14 +296,14 @@
     <visual>
       <geometry>
-        <cylinder length="${polelen}" radius="0.01"/>
-      </geometry>
-      <origin xyz="${polelen/2} 0 0" rpy="0 ${pi/2} 0 "/>
+        <cylinder length="${polelength}" radius="0.01"/>
+      </geometry>
+      <origin xyz="${polelength/2} 0 0" rpy="0 ${pi/2} 0 "/>
       <material name="green"/>
     </visual>
     <collision>
       <geometry>
-        <cylinder length="${polelen}" radius="0.01"/>
-      </geometry>
-      <origin xyz="${polelen/2} 0 0" rpy="0 0 0 "/>
+        <cylinder length="${polelength}" radius="0.01"/>
+      </geometry>
+      <origin xyz="${polelength/2} 0 0" rpy="0 0 0 "/>
     </collision>
     <xacro:default_inertial mass="0.05"/>
@@ -313,5 +313,5 @@
       <axis xyz="0 0 ${reflect}"/>
       <limit effort="1000.0" lower="0.0" upper="0.548" velocity="0.5"/>
-      <origin rpy="0 0 0" xyz="${polelen} ${reflect*0.01} 0"/>
+      <origin rpy="0 0 0" xyz="${polelength} ${reflect*0.01} 0"/>
       <parent link="gripper_pole"/>
       <child link="${prefix}_gripper"/>
