Commit message: torso link working

File: src/martin_bot/urdf/martin_bot.xacro (robot description, xacro)
@@ -3,11 +3,11 @@
   <xacro:property name="chassissize"       value=".4 .4 .1" />
   <xacro:property name="chassispose"       value="0 0 0.1 0 0 0" />
-  <xacro:property name="chassisorigin"     value="0.0 0.0 0.06" />
+  <xacro:property name="chassisorigin"     value="0.0 0.0 0.0" />
   <xacro:property name="wheelradius"       value="0.1" />
   <xacro:property name="wheellength"       value="0.05" />
   <xacro:property name="leftwheelorigin"   value="0.0  0.0 0.0" />
   <xacro:property name="rightwheelorigin"  value="0.0  0.0 0.0" />
-  <xacro:property name="leftwheelhinge"    value="0 0.25 0" />
-  <xacro:property name="rightwheelhinge"   value="0 -0.25 0" />
+  <xacro:property name="leftwheelhinge"    value="0 0.23 0" />
+  <xacro:property name="rightwheelhinge"   value="0 -0.23 0" />
   <xacro:property name="casterradius"      value="0.05" />
   <xacro:property name="frontcasterorigin" value="-0.15 0 -0.05" />
@@ -18,5 +18,6 @@
   <xacro:property name="torsoradius"       value="0.1" />
   <xacro:property name="torsolength"       value="0.2" />
-  <xacro:property name="torsoorigin"       value="0.0 0.0 0.1" />
+  <xacro:property name="torsoorigin"       value="0.0 0.0 0.0" />
+  <xacro:property name="torsolink"         value="0.0 0.0 0.1" />
   <xacro:property name="polelength"        value="0.3" />
   <xacro:property name="width"             value="0.2" />
@@ -54,5 +55,51 @@
       <material name="red"/>
    </visual>
-    <collision name='torsocollision'>
+    <collision name='back_caster_collision'>
+      <origin xyz="${backcasterorigin}" rpy=" 0 0 0"/>
+      <geometry>
+        <sphere radius="${casterradius}"/>
+      </geometry>
+      <surface>
+        <friction>
+          <ode>
+            <mu>0</mu>
+            <mu2>0</mu2>
+            <slip1>1.0</slip1>
+            <slip2>1.0</slip2>
+          </ode>
+        </friction>
+      </surface>
+    </collision>
+    <visual name='back_caster_visual'>
+      <origin xyz="${backcasterorigin}" rpy=" 0 0 0"/>
+      <geometry>
+        <sphere radius="0.05"/>
+      </geometry>
+    </visual>
+    <collision name='front_caster_collision'>
+      <origin xyz="${frontcasterorigin}" rpy=" 0 0 0"/>
+      <geometry>
+        <sphere radius="${casterradius}"/>
+      </geometry>
+      <surface>
+        <friction>
+          <ode>
+            <mu>0</mu>
+            <mu2>0</mu2>
+            <slip1>1.0</slip1>
+            <slip2>1.0</slip2>
+          </ode>
+        </friction>
+      </surface>
+    </collision>
+    <visual name='front_caster_visual'>
+      <origin xyz="${frontcasterorigin}" rpy=" 0 0 0"/>
+      <geometry>
+        <sphere radius="${casterradius}"/>
+      </geometry>
+    </visual>
+  </link>
+	<link name="torso">
+	 <collision name='torsocollision'>
       <origin xyz="${torsoorigin}" rpy=" 0 0 0"/>
       <geometry>
@@ -60,4 +107,13 @@
       </geometry>
     </collision>
+		 <inertial>
+      <mass value="5.0"/>
+      <origin xyz="${torsoorigin}" rpy=" 0 0 0"/>
+      <inertia
+          ixx="0.1" ixy="0" ixz="0"
+          iyy="0.1" iyz="0"
+          izz="0.1"
+      />
+    </inertial>
     <visual name='torso_visual'>
       <origin xyz="${torsoorigin}" rpy=" 0 0 0"/>
@@ -65,51 +121,15 @@
           <cylinder radius="${torsoradius}" length="${torsolength}"/>
       </geometry>
-      <material name="green"/>
+      <material name="black"/>
    </visual>
-    <collision name='back_caster_collision'>
-      <origin xyz="${backcasterorigin}" rpy=" 0 0 0"/>
-      <geometry>
-        <sphere radius="${casterradius}"/>
-      </geometry>
-      <surface>
-        <friction>
-          <ode>
-            <mu>0</mu>
-            <mu2>0</mu2>
-            <slip1>1.0</slip1>
-            <slip2>1.0</slip2>
-          </ode>
-        </friction>
-      </surface>
-    </collision>
-    <visual name='back_caster_visual'>
-      <origin xyz="${backcasterorigin}" rpy=" 0 0 0"/>
-      <geometry>
-        <sphere radius="0.05"/>
-      </geometry>
-    </visual>
-    <collision name='front_caster_collision'>
-      <origin xyz="${frontcasterorigin}" rpy=" 0 0 0"/>
-      <geometry>
-        <sphere radius="${casterradius}"/>
-      </geometry>
-      <surface>
-        <friction>
-          <ode>
-            <mu>0</mu>
-            <mu2>0</mu2>
-            <slip1>1.0</slip1>
-            <slip2>1.0</slip2>
-          </ode>
-        </friction>
-      </surface>
-    </collision>
-    <visual name='front_caster_visual'>
-      <origin xyz="${frontcasterorigin}" rpy=" 0 0 0"/>
-      <geometry>
-        <sphere radius="${casterradius}"/>
-      </geometry>
-    </visual>
-  </link>
+	</link>
+	<joint type="continuous" name="torsolink">
+    <origin xyz="${torsolink}" rpy="0 0 0"/>
+    <child link="torso"/>
+    <parent link="chassis"/>
+    <axis xyz="0 0 1" rpy="0 0 0"/>
+    <limit effort="10000" velocity="1000"/>
+    <joint_properties damping="1.0" friction="1.0"/>
+  </joint>
   <link name="left_wheel">
     <collision name='left_wheel_collision'>

Commit message: first pr2 gripper added

File: src/martin_bot/urdf/martin_bot.xacro (robot description, xacro)
@@ -16,10 +16,10 @@
 	<xacro:property name="cameraorigin"      value="0.0 0.0 0.0" />
 	<xacro:property name="hokuyoorigin"      value="0.0 0.0 0.0" />
+  <xacro:property name="torsolink"         value="0.0 0.0 0.1" />
   <xacro:property name="torsoradius"       value="0.1" />
   <xacro:property name="torsolength"       value="0.2" />
   <xacro:property name="torsoorigin"       value="0.0 0.0 0.0" />
-  <xacro:property name="torsolink"         value="0.0 0.0 0.1" />
   <xacro:property name="polelength"        value="0.3" />
-  <xacro:property name="width"             value="0.2" />
+  <xacro:property name="width"             value="0.15" />
   <xacro:include filename="$(find martin_bot)/urdf/martin_bot.gazebo" />
 	<!-- Import Rviz colors -->
@@ -305,6 +305,8 @@
     </inertial>
   </xacro:macro>
+	<!-- Grippers -->
   <joint name="gripper_extension" type="prismatic">
-    <parent link="robot_footprint"/>
+		<origin xyz="0.0 0.07 0.08" rpy="0 0 0"/>
+    <parent link="torso"/>
     <child link="gripper_pole"/>
     <limit effort="1000.0" lower="-${width*2-.02}" upper="0" velocity="0.5"/>
@@ -313,5 +315,5 @@
     <dynamics damping="1.0" friction="1.0"/>
   </joint>
-  <link name="gripper_pole">
+	<link name="gripper_pole">
     <visual>
       <geometry>
@@ -339,5 +341,5 @@
       <dynamics damping="0.0" friction="0.0"/>
     </joint>
-    <link name="${prefix}_gripper">
+		<link name="${prefix}_gripper">
       <visual>
         <origin rpy="${(reflect-1)/2*pi} 0 0" xyz="0 0 0"/>

Commit message: finished martin_bot

File: src/martin_bot/urdf/martin_bot.xacro (robot description, xacro)
@@ -20,5 +20,5 @@
   <xacro:property name="torsolength"       value="0.2" />
   <xacro:property name="torsoorigin"       value="0.0 0.0 0.0" />
-  <xacro:property name="polelength"        value="0.3" />
+  <xacro:property name="polelength"        value="0.2" />
   <xacro:property name="width"             value="0.15" />
   <xacro:include filename="$(find martin_bot)/urdf/martin_bot.gazebo" />
@@ -305,9 +305,9 @@
     </inertial>
   </xacro:macro>
-	<!-- Grippers -->
-  <joint name="gripper_extension" type="prismatic">
-		<origin xyz="0.0 0.07 0.08" rpy="0 0 0"/>
+	<!-- Gripper1 (left) -->
+  <joint name="gripper_extension1" type="prismatic">
+		<origin xyz="0.0 0.09 0.08" rpy="0 0 0"/>
     <parent link="torso"/>
-    <child link="gripper_pole"/>
+    <child link="gripper_pole1"/>
     <limit effort="1000.0" lower="-${width*2-.02}" upper="0" velocity="0.5"/>
     <origin rpy="0 0 0" xyz="0 0 0.15"/>
@@ -315,5 +315,5 @@
     <dynamics damping="1.0" friction="1.0"/>
   </joint>
-	<link name="gripper_pole">
+	<link name="gripper_pole1">
     <visual>
       <geometry>
@@ -321,5 +321,5 @@
       </geometry>
       <origin xyz="${polelength/2} 0 0" rpy="0 ${pi/2} 0 "/>
-      <material name="green"/>
+      <material name="grey"/>
     </visual>
     <collision>
@@ -331,15 +331,15 @@
     <xacro:default_inertial mass="0.05"/>
   </link>
-  <xacro:macro name="gripper" params="prefix reflect">
-    <joint name="${prefix}_gripper_joint" type="revolute">
+  <xacro:macro name="gripper1" params="prefix reflect">
+    <joint name="${prefix}_gripper_joint1" type="revolute">
       <axis xyz="0 0 ${reflect}"/>
       <limit effort="1000.0" lower="0.0" upper="0.548" velocity="0.5"/>
       <origin rpy="0 0 0" xyz="${polelength} ${reflect*0.01} 0"/>
-      <parent link="gripper_pole"/>
-      <child link="${prefix}_gripper"/>
+      <parent link="gripper_pole1"/>
+      <child link="${prefix}_gripper1"/>
       <limit effort="30" velocity="1.0"/>
       <dynamics damping="0.0" friction="0.0"/>
     </joint>
-		<link name="${prefix}_gripper">
+		<link name="${prefix}_gripper1">
       <visual>
         <origin rpy="${(reflect-1)/2*pi} 0 0" xyz="0 0 0"/>
@@ -356,9 +356,9 @@
       <xacro:default_inertial mass="0.05"/>
     </link>
-    <joint name="${prefix}_tip_joint" type="fixed">
-      <parent link="${prefix}_gripper"/>
-      <child link="${prefix}_tip"/>
+    <joint name="${prefix}_tip_joint1" type="fixed">
+      <parent link="${prefix}_gripper1"/>
+      <child link="${prefix}_tip1"/>
     </joint>
-    <link name="${prefix}_tip">
+    <link name="${prefix}_tip1">
       <visual>
         <origin rpy="${(reflect-1)/2*pi} 0 0" xyz="0.09137 0.00495 0"/>
@@ -376,5 +376,78 @@
     </link>
   </xacro:macro>
-  <xacro:gripper prefix="left" reflect="1" />
-  <xacro:gripper prefix="right" reflect="-1" />
+<!-- Gripper2 (Right) -->
+  <joint name="gripper_extension2" type="prismatic">
+		<origin xyz="0.0 -0.09 0.08" rpy="0 0 0"/>
+    <parent link="torso"/>
+    <child link="gripper_pole2"/>
+    <limit effort="1000.0" lower="-${width*2-.02}" upper="0" velocity="0.5"/>
+    <origin rpy="0 0 0" xyz="0 0 0.15"/>
+    <limit effort="30" velocity="0.2"/>
+    <dynamics damping="1.0" friction="1.0"/>
+  </joint>
+	<link name="gripper_pole2">
+    <visual>
+      <geometry>
+        <cylinder length="${polelength}" radius="0.01"/>
+      </geometry>
+      <origin xyz="${polelength/2} 0 0" rpy="0 ${pi/2} 0 "/>
+      <material name="grey"/>
+    </visual>
+    <collision>
+      <geometry>
+        <cylinder length="${polelength}" radius="0.01"/>
+      </geometry>
+      <origin xyz="${polelength/2} 0 0" rpy="0 0 0 "/>
+    </collision>
+    <xacro:default_inertial mass="0.05"/>
+  </link>
+  <xacro:macro name="gripper2" params="prefix reflect">
+    <joint name="${prefix}_gripper_joint2" type="revolute">
+      <axis xyz="0 0 ${reflect}"/>
+      <limit effort="1000.0" lower="0.0" upper="0.548" velocity="0.5"/>
+      <origin rpy="0 0 0" xyz="${polelength} ${reflect*0.01} 0"/>
+      <parent link="gripper_pole2"/>
+      <child link="${prefix}_gripper2"/>
+      <limit effort="30" velocity="1.0"/>
+      <dynamics damping="0.0" friction="0.0"/>
+    </joint>
+		<link name="${prefix}_gripper2">
+      <visual>
+        <origin rpy="${(reflect-1)/2*pi} 0 0" xyz="0 0 0"/>
+        <geometry>
+          <mesh filename="package://martin_bot/meshes/l_finger.dae"/>
+        </geometry>
+      </visual>
+      <collision>
+        <geometry>
+          <mesh filename="package://martin_bot/meshes/l_finger.dae"/>
+        </geometry>
+        <origin rpy="${(reflect-1)/2*pi} 0 0" xyz="0 0 0"/>
+      </collision>
+      <xacro:default_inertial mass="0.05"/>
+    </link>
+    <joint name="${prefix}_tip_joint2" type="fixed">
+      <parent link="${prefix}_gripper2"/>
+      <child link="${prefix}_tip2"/>
+    </joint>
+    <link name="${prefix}_tip2">
+      <visual>
+        <origin rpy="${(reflect-1)/2*pi} 0 0" xyz="0.09137 0.00495 0"/>
+        <geometry>
+          <mesh filename="package://martin_bot/meshes/l_finger_tip.dae"/>
+        </geometry>
+      </visual>
+      <collision>
+        <geometry>
+          <mesh filename="package://martin_bot/meshes/l_finger_tip.dae"/>
+        </geometry>
+        <origin rpy="${(reflect-1)/2*pi} 0 0" xyz="0.09137 0.00495 0"/>
+      </collision>
+      <xacro:default_inertial mass="0.05"/>
+    </link>
+  </xacro:macro>
+  <xacro:gripper1 prefix="left" reflect="1" />
+  <xacro:gripper1 prefix="right" reflect="-1" />
+	<xacro:gripper2 prefix="left" reflect="1" />
+  <xacro:gripper2 prefix="right" reflect="-1" />
 </robot>

Commit message: working solution

File: src/martin_bot/urdf/martin_bot.xacro (robot description, xacro)
@@ -20,5 +20,5 @@
   <xacro:property name="torsolength"       value="0.2" />
   <xacro:property name="torsoorigin"       value="0.0 0.0 0.0" />
-  <xacro:property name="polelength"        value="0.2" />
+  <xacro:property name="polelength"        value="0.1" />
   <xacro:property name="width"             value="0.15" />
   <xacro:include filename="$(find martin_bot)/urdf/martin_bot.gazebo" />
@@ -124,5 +124,5 @@
    </visual>
 	</link>
-	<joint type="continuous" name="torsolink">
+	<joint name="torsolink" type="fixed">
     <origin xyz="${torsolink}" rpy="0 0 0"/>
     <child link="torso"/>
@@ -307,5 +307,5 @@
 	<!-- Gripper1 (left) -->
   <joint name="gripper_extension1" type="prismatic">
-		<origin xyz="0.0 0.09 0.08" rpy="0 0 0"/>
+		<origin xyz="0.0 0.09 0.07" rpy="0 0 0"/>
     <parent link="torso"/>
     <child link="gripper_pole1"/>
@@ -378,5 +378,5 @@
 <!-- Gripper2 (Right) -->
   <joint name="gripper_extension2" type="prismatic">
-		<origin xyz="0.0 -0.09 0.08" rpy="0 0 0"/>
+		<origin xyz="0.0 -0.09 0.07" rpy="0 0 0"/>
     <parent link="torso"/>
     <child link="gripper_pole2"/>
